File: teclado46_stm32.kicad_pcb (KiCad board)
At the start: 2 copper layers, 228.6 x 76.2 mm, 104 parts, among them J2 78171-0004, U1 XC6206PxxxMR, U2 STM32G474CETx, U4 W25Q128JVS

Commit message: chore: add boot0 and nrst
Parts:
- removed C14: 1u, Capacitor_SMD:C_0402_1005Metric
- removed U4: W25Q128JVS, Package_SO:SOIC-8_5.3x5.3mm_P1.27mm
- U2: value STM32G474CETx -> STM32G0B1RETx; footprint Package_QFP:LQFP-48_7x7mm_P0.5mm -> Package_QFP:LQFP-64_10x10mm_P0.5mm
- moved MX1 409.3 mm to (441.1, 32.9)
- moved MX13 394.4 mm to (423.9, 93.1)
- moved MX2 390.6 mm to (441.1, 47.9)
- moved MX14 377.5 mm to (423.9, 108.1)
- moved MX3 372.5 mm to (441.1, 63.0)
- moved MX15 361.4 mm to (423.9, 123.2)
- moved MX25 359.8 mm to (389.6, 32.9)
- moved MX4 355.2 mm to (441.1, 78.0)
- moved J2 347.1 mm to (444.7, 165.5)
- moved MX16 346.2 mm to (423.9, 138.2)
- moved U1 344.9 mm to (437.8, 164.6), turned to 180 degrees
- moved MX37 340.8 mm to (372.5, 93.1)
- moved MX26 339.5 mm to (389.6, 47.9)
- moved MX5 338.7 mm to (441.1, 93.1)
- moved C2 337.9 mm to (433.1, 150.7)
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Connections:
- C3 pad 2: GND -> Net-(C3-Pad2)
- C4 pad 2: GND -> Net-(C3-Pad2)
- C5 pad 2: GND -> Net-(C3-Pad2)
- C6 pad 2: GND -> Net-(C3-Pad2)
- C7 pad 2: GND -> Net-(C3-Pad2)
- U2 pad 10: Q_SEL -> unconnected-(U2-PF0-Pad10)
- U2 pad 11: Q_CLK -> unconnected-(U2-PF1-Pad11)
- U2 pad 12: unconnected-(U2-PA4-Pad12) -> NRST
- U2 pad 14: Q_103 -> unconnected-(U2-PC1-Pad14)
- U2 pad 15: Q_102 -> unconnected-(U2-PC2-Pad15)
- U2 pad 16: Q_101 -> unconnected-(U2-PC3-Pad16)
- U2 pad 17: Q_100 -> unconnected-(U2-PA0-Pad17)
- U2 pad 18: ROW 3 -> unconnected-(U2-PA1-Pad18)
- U2 pad 19: GND -> unconnected-(U2-PA2-Pad19)
- U2 pad 21: +3V3 -> unconnected-(U2-PA4-Pad21)
- U2 pad 23: GND -> unconnected-(U2-PA6-Pad23)
- U2 pad 24: +3V3 -> unconnected-(U2-PA7-Pad24)
- U2 pad 25: COL 0 -> unconnected-(U2-PC4-Pad25)
- U2 pad 26: COL 1 -> unconnected-(U2-PC5-Pad26)
- U2 pad 27: COL 2 -> unconnected-(U2-PB0-Pad27)
- U2 pad 28: COL 3 -> unconnected-(U2-PB1-Pad28)
- U2 pad 29: COL 4 -> unconnected-(U2-PB2-Pad29)
- U2 pad 30: COL 5 -> unconnected-(U2-PB10-Pad30)
- U2 pad 33: D- -> unconnected-(U2-PB13-Pad33)
- U2 pad 34: D+ -> unconnected-(U2-PB14-Pad34)
- U2 pad 35: GND -> unconnected-(U2-PB15-Pad35)
- U2 pad 36: +3V3 -> unconnected-(U2-PA8-Pad36)
- U2 pad 37: ROW 2 -> unconnected-(U2-PA9/UCPD1_DBCC1-Pad37)
- U2 pad 4: COL 7 -> unconnected-(U2-PC14-Pad4)
- U2 pad 42: ROW 1 -> unconnected-(U2-PA10/UCPD1_DBCC2-Pad42)
- U2 pad 43: ROW 0 -> D-
- U2 pad 44: COL 6 -> D+
- U2 pad 45: BOOT0 -> unconnected-(U2-PA13-Pad45)
- U2 pad 46: unconnected-(U2-PB9-Pad46) -> BOOT0
- U2 pad 47: GND -> unconnected-(U2-PA15-Pad47)
- U2 pad 48: +3V3 -> unconnected-(U2-PC8-Pad48)
- U2 pad 5: COL 8 -> unconnected-(U2-PC15-Pad5)
- U2 pad 6: COL 9 -> unconnected-(U2-VBAT-Pad6)
- U2 pad 7: NRST -> unconnected-(U2-VREF+-Pad7)
- U2 pad 8: COL 10 -> +3V3
- U2 pad 9: COL 11 -> GND
Routing:
- net ROW 0: track 254.1 -> 0.00 mm, vias 2 -> 0
- net ROW 1: track 234.8 -> 0.00 mm
- net ROW 3: track 218.8 -> 0.00 mm, vias 3 -> 0
- net ROW 2: track 217.9 -> 0.00 mm, vias 2 -> 0
- net COL 0: track 172.7 -> 0.00 mm
- net COL 11: track 158.1 -> 0.00 mm
- net COL 1: track 153.5 -> 0.00 mm
- net COL 10: track 136.5 -> 0.00 mm
- net COL 2: track 134.8 -> 0.00 mm
- net COL 9: track 117.9 -> 0.00 mm
- net COL 3: track 115.5 -> 0.00 mm
- net COL 8: track 100.1 -> 0.00 mm
- net COL 4: track 89.7 -> 0.00 mm
- net +3V3: track 70.1 -> 0.00 mm
- net COL 7: track 69.7 -> 0.00 mm
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- removed copper zone on B.Cu, net GND
- removed copper zone on F.Cu, net GND
Other:
- board outline removed
