File: matrix.kicad_sch (KiCad schematic)
At the start: 92 parts

Commit message: chore: wired matrix schematic
Connections:
- net COL 3: now reaches MX40.1
- net COL 3: now also MX16.1, MX28.1, MX4.1
- net ROW 3: now reaches D42.1 (K)
- net ROW 3: now also D37.1 (K), D38.1 (K), D39.1 (K), D40.1 (K), D41.1 (K), D43.1 (K), D44.1 (K), D45.1 (K), D46.1 (K)
- net COL 9: now reaches MX44.1
- net COL 9: now also MX10.1, MX22.1, MX34.1
- net ROW 0: now reaches D10.1 (K)
- net ROW 0: now also D1.1 (K), D11.1 (K), D12.1 (K), D2.1 (K), D3.1 (K), D4.1 (K), D5.1 (K), D6.1 (K), D7.1 (K), D8.1 (K), D9.1 (K)
- net ROW 2: now reaches D33.1 (K)
- net ROW 2: now also D25.1 (K), D26.1 (K), D27.1 (K), D28.1 (K), D29.1 (K), D30.1 (K), D31.1 (K), D32.1 (K), D34.1 (K), D35.1 (K), D36.1 (K)
- net COL 6: now reaches MX31.1
- net COL 6: now also MX19.1, MX7.1
- net ROW 1: now reaches D20.1 (K)
- net ROW 1: now also D13.1 (K), D14.1 (K), D15.1 (K), D16.1 (K), D17.1 (K), D18.1 (K), D19.1 (K), D21.1 (K), D22.1 (K), D23.1 (K), D24.1 (K)
- net COL 2: now reaches MX27.1
- net COL 2: now also MX15.1, MX3.1, MX39.1
- net COL 4: now reaches MX17.1
- net COL 4: now also MX29.1, MX41.1, MX5.1
- net COL 8: now reaches MX9.1
- net COL 8: now also MX21.1, MX33.1, MX43.1
- net COL 0: now reaches MX13.1
- net COL 0: now also MX1.1, MX25.1, MX37.1
- net COL 1: now reaches MX2.1
- net COL 1: now also MX14.1, MX26.1, MX38.1
- net COL 7: now reaches MX32.1
- net COL 7: now also MX20.1, MX42.1, MX8.1
- net COL 11: now reaches MX46.1
- net COL 11: now also MX12.1, MX24.1, MX36.1
- net COL 10: now reaches MX45.1
- net COL 10: now also MX11.1, MX23.1, MX35.1
- net COL 5: now reaches MX6.1
- net COL 5: now also MX18.1, MX30.1

Commit message: chore: add stabs
Parts:
- added S1, S2: MX_stab, PCM_marbastlib-mx:STAB_MX_P_2u, symbol PCM_marbastlib-mx:MX_stab
Changed lines of the file:
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@@
+	)
+	(symbol
+		(lib_id "PCM_marbastlib-mx:MX_stab")
+		(at 101.6 139.7 0)
+		(unit 1)
+		(exclude_from_sim no)
+		(in_bom yes)
+		(on_board yes)
+		(dnp no)
+		(fields_autoplaced yes)
+		(property "Reference" "S1"
+			(at 107.95 138.3029 0)
+			(effects
+				(font
+					(size 1.27 1.27)
+				)
+				(justify left)
+			)
+		)
+		(property "Value" "MX_stab"
+			(at 107.95 140.8429 0)
+			(effects
+				(font
+					(size 1.27 1.27)
+				)
+				(justify left)
+			)
+		)
+		(property "Footprint" "PCM_marbastlib-mx:STAB_MX_P_2u"
+			(at 101.6 139.7 0)
+			(effects
+				(font
+					(size 1.27 1.27)
+				)
+				(hide yes)
+			)
+		)
+		(property "Datasheet" ""
+			(at 101.6 139.7 0)
+			(effects
+				(font
+					(size 1.27 1.27)
+				)
+				(hide yes)
+			)
+		)
+		(property "Description" "Cherry MX-style stabilizer"
+			(at 101.6 139.7 0)
+			(effects
+				(font
+					(size 1.27 1.27)
+				)
+				(hide yes)
+			)
+		)
+		(instances
+			(project ""
+				(path "/6ed4739c-92e8-425a-abb0-74006c04cb3a/77b5a20e-1b3c-475a-a3a6-da7292e51f2c"
+					(reference "S1")
+					(unit 1)
+				)
+			)
+		)
 	)
 	(symbol
@@
 					(unit 1)
 				)
+			)
+		)
+	)
+	(symbol
+		(lib_id "PCM_marbastlib-mx:MX_stab")
+		(at 127 139.7 0)
+		(unit 1)
+		(exclude_from_sim no)
+		(in_bom yes)
+		(on_board yes)
+		(dnp no)
+		(fields_autoplaced yes)
+		(property "Reference" "S2"
+			(at 133.35 138.3029 0)
+			(effects
+				(font
+					(size 1.27 1.27)
+				)
+				(justify left)
+			)
+		)
+		(property "Value" "MX_stab"
+			(at 133.35 140.8429 0)
+			(effects
+				(font
+					(size 1.27 1.27)
+				)
+				(justify left)
+			)
+		)
+		(property "Footprint" "PCM_marbastlib-mx:STAB_MX_P_2u"
+			(at 127 139.7 0)
+			(effects
+				(font
+					(size 1.27 1.27)
+				)
+				(hide yes)
+			)
+		)
+		(property "Datasheet" ""
+			(at 127 139.7 0)
+			(effects
+				(font
+					(size 1.27 1.27)
+				)
+				(hide yes)
+			)
+		)
+		(property "Description" "Cherry MX-style stabilizer"
+			(at 127 139.7 0)
+			(effects
+				(font
+					(size 1.27 1.27)
+				)
+				(hide yes)
+			)
+		)
+		(instances
+			(project "teclado46_stm32"
+				(path "/6ed4739c-92e8-425a-abb0-74006c04cb3a/77b5a20e-1b3c-475a-a3a6-da7292e51f2c"
+					(reference "S2")
+					(unit 1)
+				)
